Commit message: add option to load four cams instead of 5

File: urdf/alphasense.urdf.xacro (robot description, xacro)
@@ -15,5 +15,5 @@
 <!-- YAML file containing the default values from CAD -->
 <xacro:property name="default_calib" value="$(find alphasense_description)/urdf/calibrations/default_calibration.yaml" />
-<xacro:macro name="alphasense" params="parent *origin name:=alphasense calib_file:=${default_calib}">
+<xacro:macro name="alphasense" params="parent *origin name:=alphasense calib_file:=${default_calib} four_cams:=false">
 <!-- load the YAML calibration file into a property -->
 <xacro:property name="calib" value="${load_yaml(calib_file)}"/>
@@ -26,5 +26,10 @@
     <visual>
       <geometry>
-        <mesh filename="package://alphasense_description/urdf/meshes/alphasense_simplified.dae" />
+        <xacro:if value="${four_cams}">
+          <mesh filename="package://alphasense_description/urdf/meshes/alphasense_simplified_4cams.dae" />
+        </xacro:if>
+        <xacro:unless value="${four_cams}">
+          <mesh filename="package://alphasense_description/urdf/meshes/alphasense_simplified.dae" />
+        </xacro:unless>
       </geometry>
     </visual>
@@ -91,14 +96,4 @@
     </visual>
   </link>
-  <link name="cam_top">
-    <visual>
-      <geometry>
-        <box size="1e-3 1e-3 1e-3" />
-      </geometry>
-      <material name="black">
-        <color rgba="0 0 0 1" />
-      </material>
-    </visual>
-  </link>
   <!-- front right camera which is cam0 in alphasense driver -->
   <joint name="imu_to_cam_front_right_joint" type="fixed">
@@ -125,16 +120,28 @@
     <child link="cam_front_left" />
   </joint>
-  <!-- top camera which is cam2 in alphasense driver, haven't calibrated yet -->
-  <joint name="imu_to_cam_top_joint" type="fixed">
-    <!--origin xyz="-0.00789 -0.07720 -0.01356" rpy="1.5733 0.00443 -0.0052"/-->
-    <origin xyz="${calib['imu_to_cam2']['x']}
-                 ${calib['imu_to_cam2']['y']}
-                 ${calib['imu_to_cam2']['z']}"
-            rpy="${calib['imu_to_cam2']['roll']}
-                 ${calib['imu_to_cam2']['pitch']}
-                 ${calib['imu_to_cam2']['yaw']}"/>
-    <parent link="${name}_imu" />
-    <child link="cam_top" />
-  </joint>
+  <xacro:unless value="${four_cams}">
+    <link name="cam_top">
+      <visual>
+        <geometry>
+          <box size="1e-3 1e-3 1e-3" />
+        </geometry>
+        <material name="black">
+          <color rgba="0 0 0 1" />
+        </material>
+      </visual>
+    </link>
+    <!-- top camera which is cam2 in alphasense driver, haven't calibrated yet -->
+    <joint name="imu_to_cam_top_joint" type="fixed">
+      <!--origin xyz="-0.00789 -0.07720 -0.01356" rpy="1.5733 0.00443 -0.0052"/-->
+      <origin xyz="${calib['imu_to_cam2']['x']}
+                   ${calib['imu_to_cam2']['y']}
+                   ${calib['imu_to_cam2']['z']}"
+              rpy="${calib['imu_to_cam2']['roll']}
+                   ${calib['imu_to_cam2']['pitch']}
+                   ${calib['imu_to_cam2']['yaw']}"/>
+      <parent link="${name}_imu" />
+      <child link="cam_top" />
+    </joint>
+  </xacro:unless>
   <!-- side right camera which is cam3 in alphasense driver -->
   <joint name="imu_to_cam_side_right_joint" type="fixed">

File: urdf/alphasense_standalone.urdf.xacro (robot description, xacro)
@@ -14,8 +14,9 @@
 <robot name="alphasense_standalone" xmlns:xacro="http://www.ros.org/wiki/xacro">
   <xacro:arg name="calib_file" default="$(find alphasense_description)/urdf/calibrations/default_calibration.yaml"/>
+  <xacro:arg name="four_cams" default="false"/>
   <xacro:property name="calib_file" value="$(arg calib_file)"/>
   <xacro:include filename="$(find alphasense_description)/urdf/alphasense.urdf.xacro" />
   <link name="base" />
-  <xacro:alphasense parent="base" calib_file="${calib_file}">
+  <xacro:alphasense parent="base" calib_file="${calib_file}" four_cams="$(arg four_cams)">
     <origin xyz="0 0 0" rpy="0 0 0" />
   </xacro:alphasense>

Commit message: update deprecated command

File: urdf/alphasense.urdf.xacro (robot description, xacro)
@@ -17,5 +17,5 @@
 <xacro:macro name="alphasense" params="parent *origin name:=alphasense calib_file:=${default_calib} four_cams:=false">
 <!-- load the YAML calibration file into a property -->
-<xacro:property name="calib" value="${load_yaml(calib_file)}"/>
+<xacro:property name="calib" value="${xacro.load_yaml(calib_file)}"/>
 <joint name="${parent}_to_alphasense" type="fixed">
     <xacro:insert_block name="origin"/>
