Commit message: add calibration converter script

File: urdf/alphasense_standalone.urdf (robot description, URDF)
Before this commit: robot alphasense_standalone, 7 links, 6 joints
Links:
- removed link imu_link
- added link alphasense_imu; visual box size=3e-3 2e-3 1e-3
- added link cam_top; visual box size=1e-3 1e-3 1e-3
Joints:
- removed joint front_left_cam_joint
- removed joint front_right_cam_joint
- removed joint side_left_cam_joint
- removed joint side_right_cam_joint
- added joint imu_to_cam_front_left_joint: type fixed, parent alphasense_imu, child cam_front_left, origin xyz=0.05                   -0.06355                  -0.0076 rpy=1.5707963267948966                  0.0                  1.5707963267948966
- added joint imu_to_cam_front_right_joint: type fixed, parent alphasense_imu, child cam_front_right, origin xyz=0.05                   0.04645                  -0.0076 rpy=1.5707963267948966                  0.0                  1.5707963267948966
- added joint imu_to_cam_side_left_joint: type fixed, parent alphasense_imu, child cam_side_left, origin xyz=-0.0075                   -0.07804                  -0.0076 rpy=-1.5707963267948966                  3.141592653589793                  3.141592653589793
- added joint imu_to_cam_side_right_joint: type fixed, parent alphasense_imu, child cam_side_right, origin xyz=-0.0075                   0.06094                  -0.0076 rpy=1.5707963267948966                  0.0                  3.141592653589793
- added joint imu_to_cam_top_joint: type fixed, parent alphasense_imu, child cam_top, origin xyz=0.01                   -0.00855                  -0.035 rpy=3.141592653589793                  0.0                  0.0
- joint imu_joint: child imu_link -> alphasense_imu; origin xyz=6e-3 -8.55e-3 17.4e-3 rpy=3.141592653589793 0 0 -> xyz=6.0e-3 -8.55e-3 17.4e-3 rpy=3.141592653589793 0 0

File: urdf/alphasense_standalone.urdf.xacro (robot description, xacro)
@@ -13,7 +13,9 @@
 -->
 <robot name="alphasense_standalone" xmlns:xacro="http://www.ros.org/wiki/xacro">
+  <xacro:arg name="calib_file" default="$(find alphasense_description/urdf/calibrations/default_calibration.yaml"/>
+  <xacro:property name="calib_file" value="$(arg calib_file)"/>
   <xacro:include filename="$(find alphasense_description)/urdf/alphasense.urdf.xacro" />
   <link name="base" />
-  <xacro:alphasense parent="base">
+  <xacro:alphasense parent="base" calib_file="${calib_file}">
     <origin xyz="0 0 0" rpy="0 0 0" />
   </xacro:alphasense>

Commit message: update urdf

File: urdf/alphasense_standalone.urdf (robot description, URDF)
Before this commit: robot alphasense_standalone, 8 links, 7 joints
Joints:
- joint imu_to_cam_top_joint: origin xyz=0.01                   -0.00855                  -0.035 rpy=3.141592653589793                  0.0                  0.0 -> xyz=0.01                     -0.00855                    -0.035 rpy=3.141592653589793                    0.0                    0.0
