Commit message: fix: Correct wrong orientation of optical camera frame by adding camera frame and rotation around y

File: urdf/alphasense_camera_module.urdf.xacro (robot description, xacro)
@@ -30,9 +30,15 @@
       <xacro:insert_block name="origin"/>
     </joint>
+    <link name="${name}_frame"/>
+    <joint name="${imu_name}_to_${name}_frame" type="fixed">
+      <parent link="${imu_name}"/>
+      <child link="${name}_frame"/>
+      <xacro:insert_block name="imu_cam_origin"/>
+    </joint>
     <link name="${name}_optical_frame"/>
-    <joint name="${imu_name}_to_${name}_optical_frame" type="fixed">
-      <parent link="${imu_name}"/>
+    <joint name="${name}_frame_to_${name}_optical_frame" type="fixed">
+      <parent link="${name}_frame"/>
       <child link="${name}_optical_frame"/>
-      <xacro:insert_block name="imu_cam_origin"/>
+      <origin xyz="0 0 0" rpy="0 -${pi/2} 0"/>
     </joint>
   </xacro:macro>
